File: KiCAD/CPU.kicad_sch (KiCad schematic)
At the start: 29 parts

Commit message: Fix DD5 and DD22
Parts:
- removed DD5: КР1533ЛИ1, Romychs_IC_DIP:DIP-14_W7.62mm, symbol Romychs_Logic_TTL:КР1533ЛИ1
- added DD5: КР1533ЛЛ1, Romychs_IC_DIP:DIP-14_W7.62mm, symbol Romychs_Logic_TTL:КР1533ЛЛ1
Connections:
- net D4: now also DD5.9 (1)
- net D6: now also DD5.10 (2)
- net F3: now also DD5.11 (3)
- net GND: now also DD5.7 (GND)
- net S2: now also DD5.13 (2)
- net VCC: now also DD5.14 (VCC)
- net ~{CSC0}: now also DD5.1
- net ~{CSE0}: now also DD5.5 (2)
- net ~{CS_ROM1}: now also DD5.3
- net ~{ENROM}: now also DD5.2, DD5.4 (1)
- net at DD6.1: now also DD5.6 (3)
- net at DD10.6 (2): now also DD5.8 (3)
- net at DD15.3 (Q0), DD16.2: now also DD5.12 (1)
