File: KiCAD/RAM_CTR.kicad_sch (KiCad schematic)
At the start: 23 parts

Commit message: Fix DD5 and DD22
Parts:
- removed DD22: КР1533ЛИ1, Romychs_IC_DIP:DIP-14_W7.62mm, symbol Romychs_Logic_TTL:КР1533ЛИ1
- added DD22: КР1533ЛЛ1, Romychs_IC_DIP:DIP-14_W7.62mm, symbol Romychs_Logic_TTL:КР1533ЛЛ1
Connections:
- net (A15): now also DD22.6 (3)
- net 32K: now also DD22.5 (2)
- net A15: now also DD22.4 (1)
- net C5: now also DD22.1
- net GC: now also DD22.2
- net GND: now also DD22.7 (GND)
- net S1: now also DD22.9 (1)
- net SR: now also DD22.10 (2)
- net VCC: now also DD22.14 (VCC)
- net at DD23.2: now also DD22.3
- net at DD16.5 (2), DD16.9 (1): now also DD22.8 (3)
