File: KiCAD/Океан-240.2.kicad_pcb (KiCad board)
At the start: 2 copper layers, 323.3 x 178.5 mm, 285 parts, among them X1 RGB-VGA, X2 Keyboard + User IO, X3 Centronics, X4 FDD-Connector, X5 User IO

Commit message: Fix DD5 and DD22
Parts:
- added ?: , , F.Cu at (233.7, 48.2)
- added ?: , , F.Cu at (121.3, 65.1)
- added ?: , , F.Cu at (48.8, 155.1)
- added ?: , , F.Cu at (45.3, 219.9)
- added ?: , , F.Cu at (45.2, 48.2)
- added ?: , , F.Cu at (171.2, 48.2)
- added ?: , , F.Cu at (361.8, 48.1)
- added ?: , , F.Cu at (361.8, 219.9)
- added REF**: MountingHole_3.2mm_M3, MountingHole:MountingHole_3.2mm_M3, F.Cu at (121.3, 155.1)
- added REF**: MountingHole_3.2mm_M3_ISO7380_Pad, MountingHole:MountingHole_3.2mm_M3_ISO7380_Pad, F.Cu at (49.3, 65.1)
- DD22, DD5: value КР1533ЛИ1 -> КР1533ЛЛ1
- moved C49 64.6 mm to (121.3, 160.4)
- moved DD8 61.0 mm to (342.3, 178.2)
- moved R4 61.0 mm to (306.8, 180.7)
- moved R44 61.0 mm to (182.3, 112.1)
- moved R46 61.0 mm to (182.3, 126.1)
- moved C2 61.0 mm to (301.1, 180.7)
- moved C28 61.0 mm to (121.3, 213.7)
- moved C31 61.0 mm to (160.7, 190.9)
- moved C36 61.0 mm to (228.0, 190.9)
- moved C51 61.0 mm to (214.1, 154.0)
- moved C64 61.0 mm to (71.8, 99.4)
- moved C65 61.0 mm to (85.8, 99.4)
- moved C66 61.0 mm to (99.8, 99.4)
- moved C67 61.0 mm to (113.7, 99.4)
- moved DA76 61.0 mm to (238.2, 79.1)
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Routing:
- net GND: track 399.8 -> 392.7 mm
- net A15: track 202.5 -> 199.8 mm
- net MD1: track 102.4 -> 105.0 mm
- net INT: track 99.7 -> 97.6 mm
- net ~{CSE0}: track 215.6 -> 217.4 mm
- net D5: track 282.8 -> 284.1 mm
- net D4: track 331.0 -> 332.2 mm
- net VR: track 329.5 -> 330.3 mm
- net A0: track 276.6 -> 275.9 mm
- net P0-PA0: track 38.6 -> 39.3 mm
- net MD0: track 99.9 -> 100.5 mm
- net ~{ENROM}: track 130.3 -> 129.7 mm
- net RST_6: track 58.9 -> 58.3 mm
- net RST3: track 132.2 -> 132.7 mm
Other:
- board size 323.3 x 178.5 mm -> 323.3 x 178.7 mm
- board text added: "v1.0.3 2026.03.10"
- board text removed: "v1.0.2 2025.12.10"
